File: PCB/BridgeWriter_v0/BridgeWriter_v0.kicad_sch (KiCad schematic)
At the start: 195 parts, among them J1 USB_B, J10 Conn_01x04, J17 Conn_01x01, J18 Conn_01x01, J2 RJ45_Bel_SI-60062-F, J24 Conn_01x04, J25 Conn_01x04, J3 Conn_01x05, J4 Conn_01x06, J6 Conn_01x04, J7 Conn_01x04, J9 Micro_SD_Card_Det2, SW1 SW_Push, SW10 SW_Push, SW2 BOOT_MODE0, SW3 SW_Push, SW4 SW_Push, SW5 SW_Push, SW6 SW_Push, SW7 SW_Push, SW8 BOOT_MODE1, SW9 SW_Push, U1 STM32H723VGTx, U10 ADP3338AKCZ-3.3, U11 OKL-T/6-W12N-C, U2 W6300, U3 ESP32-C5-WROOM-1, U5 MCP2562-E-SN, U6 MCP2562-E-SN, U7 USB3343, U8 ADP3338AKCZ-3.3, U9 CH213K, Y1 FC2012SN 32.768K-70NNA0KC0, Y2 XRCGB25M000FFS1AR0, Y3 ECS-600-8-36B-CTN-TR

Commit message: change
Parts:
- removed C25, C26: 0.1uF, Capacitor_SMD:C_0603_1608Metric_Pad1.08x0.95mm_HandSolder, symbol Device:C_Small
- removed J10: Conn_01x04, Connector_PinSocket_2.54mm:PinSocket_1x04_P2.54mm_Vertical, symbol Connector_Generic:Conn_01x04
- added U12: PT86-091940LMR, My_Library:PT86-091940LMR, symbol My_Library:PT86-091940LMR
- added U4: TLP293, Package_SO:SOIC-4_4.55x2.6mm_P1.27mm, symbol Isolator:TLP293
- R55: value 80k -> 10k
- R56: value 10k -> 1k
Connections:
- net +3.3V: now also J3.5 (Pin_5), R56.2; no longer J3.4 (Pin_4)
- net GND: now also J3.4 (Pin_4), U4.2; no longer J3.5 (Pin_5), R56.2
- net POWER_MONITOR: now also U4.3; no longer R55.2, R56.1
- net SWCLK: now also J3.2 (Pin_2); no longer J3.3 (Pin_3)
- net SWDIO: now also J3.3 (Pin_3); no longer J3.2 (Pin_2)
- net LPUART_RXD: no longer names the net of U1.69 (PA10)
- net LPUART_TXD: no longer names the net of U1.68 (PA9)
- new net: R55.2, U4.1
- new net: R56.1, U4.4
- no-connect marks 23 -> 24
Other:
- note removed: "LPUART"
- moved on the sheet: R55

Commit message: All the wiring except the power is probably done.
Parts:
- removed C1: 1uF, Capacitor_SMD:C_0603_1608Metric_Pad1.08x0.95mm_HandSolder, symbol Device:C_Small
- removed D16, D38, D39: O, LED_SMD:LED_0603_1608Metric_Pad1.05x0.95mm_HandSolder, symbol Device:LED
- removed D17, D20, D7: G, LED_SMD:LED_0603_1608Metric_Pad1.05x0.95mm_HandSolder, symbol Device:LED
- removed D4, D8: W, LED_SMD:LED_0603_1608Metric_Pad1.05x0.95mm_HandSolder, symbol Device:LED
- removed D44: LED, LED_SMD:LED_0603_1608Metric_Pad1.05x0.95mm_HandSolder, symbol Device:LED
- removed R16, R28, R29, R48, R49, R52: 1k, Resistor_SMD:R_0603_1608Metric_Pad0.98x0.95mm_HandSolder, symbol Device:R_Small
- added C25, C26, C66, C67, C68: 0.1uF, Capacitor_SMD:C_0603_1608Metric_Pad1.08x0.95mm_HandSolder, symbol Device:C_Small
- added J5, J8: Conn_01x02, Connector_JST:JST_ZH_B2B-ZR_1x02_P1.50mm_Vertical, symbol Connector_Generic:Conn_01x02
- added R59, R60: 330, Resistor_SMD:R_0603_1608Metric_Pad0.98x0.95mm_HandSolder, symbol Device:R_Small
- added R61, R62, R64: 1k, Resistor_SMD:R_0603_1608Metric_Pad0.98x0.95mm_HandSolder, symbol Device:R_Small
- added R63: 10k, Resistor_SMD:R_0603_1608Metric_Pad0.98x0.95mm_HandSolder, symbol Device:R_Small
- added U13, U14: AM8068, Package_TO_SOT_SMD:TSOT-23-6_HandSoldering, symbol My_Library:AM8068
- added U15, U16: MCP9700x-ETT, Package_TO_SOT_SMD:SOT-23, symbol Sensor_Temperature:MCP9700x-ETT
- D15, D19, D22, D24, D26, D30: value B -> G
Connections:
- net Ethernet_Active is gone; now on net FAN_INB_STM: R24.1
- net USB_Active is gone; now on net FAN_INA_STM: R32.1
- net +3.3V: now also R19.1, R20.1, R21.1, R22.1, R23.1, R61.1, R62.1; no longer SW2.1 (A), SW3.1, SW4.1, SW5.1, SW6.1, SW7.1, SW8.2 (B)
- net +5V: now also U13.4 (VCC), U14.4 (VCC), U15.1 (V_{DD}), U16.1 (V_{DD})
- net DEBUG_LED: now also U1.82 (PD1)
- net ERROR_LED: now also U1.81 (PD0)
- net Ethernet_RESET: now also U1.55 (PD8), C68.1; no longer R21.1
- net Ethernet_RX: now also U1.63 (PC6)
- net Ethernet_TX: now also U1.62 (PD15)
- net FDCAN1_RESET: now also U1.57 (PD10), C66.1; no longer R23.1
- net FDCAN1_RX: now also U1.98 (PE1)
- net FDCAN1_TX: now also U1.5 (PE6)
- net FDCAN2_RESET: now also U1.56 (PD9), C67.1; no longer R22.1
- net FDCAN2_RX: now also U1.1 (PE2)
- net FDCAN2_TX: now also U1.4 (PE5)
- net GND: now also R24.2, R32.2, R45.2, C25.2, C26.2, C66.2, C67.2, C68.2, R63.2, R64.2, U13.2 (GND), U14.2 (GND), U15.3 (GND), U16.3 (GND); no longer R19.2, R20.2, R21.2, R22.2, R23.2
- net PGOOD: now also U1.69 (PA10); no longer R45.1
- net POWER_MONITOR: now also U1.64 (PC7)
- net SDMMC_CHECK: now also U1.24 (PA2)
- net SDMMC_READ: now also U1.22 (PA0)
- net SDMMC_WRITE: now also U1.23 (PA1)
- net USB3343_RESETB: now also U1.45 (PE15)
- net USB_RESET: now also U1.54 (PB15), C26.1; no longer R20.1
- net USB_RX: now also U1.61 (PD14)
- net USB_TX: now also U1.58 (PD11)
- net W6300_ACT: now also U1.32 (PC4)
- net W6300_COL: now also U1.33 (PC5)
- net W6300_DPX: now also U1.31 (PA7)
- net W6300_INT: now also U1.42 (PE12)
- net W6300_LNK: now also U1.28 (PA4)
- net W6300_RST: now also U1.43 (PE13)
- net W6300_SPD: now also U1.30 (PA6)
- net WRITER_MODE: now also U1.84 (PD3)
- net Wi-Fi_RESET: now also U1.53 (PB14), C25.1; no longer R19.1
- net Th_ESP: now reaches U3.7 (IO1)
- net Th_ESP: now also U15.2 (V_{OUT})
- net Th_STM: now reaches U1.16 (PC1)
- net Th_STM: now also U16.2 (V_{OUT})
- net Speaker_In2: now reaches U1.2 (PE3)
- net Speaker_In2: now also R59.1
- net Speaker_In1: now reaches U1.3 (PE4)
- net Speaker_In1: now also R60.1
- net BOOTMODE: now reaches U1.44 (PE14)
- net BOOTMODE: now also SW8.2 (B)
- net FAN_INB_STM: now reaches U1.67 (PA8)
- net FAN_INB_STM: now also U13.5 (IN_B)
- net FAN_INA_STM: now reaches U1.68 (PA9)
- net FAN_INA_STM: now also U13.6 (IN_A)
- net at U12.1 (In): now also R60.2
- net at U12.2 (In): now also R59.2
- net FLASH_USERCODE: no longer names the net of SW8.3 (C)
- net FLASH_USERCODE: now also R63.1
- net RAM_BOOTLOADER: no longer names the net of SW8.1 (A)
- net RAM_BOOTLOADER: now also R62.2
- new net: R21.2, SW4.1
- new net: R23.2, SW2.1 (A)
- new net: J8.1 (Pin_1), U14.1 (OUT_A)
- new net: J8.2 (Pin_2), U14.3 (OUT_B)
- new net: R19.2, SW6.1
- new net: R20.2, SW5.1
- new net: J5.1 (Pin_1), U13.1 (OUT_A)
- new net: J5.2 (Pin_2), U13.3 (OUT_B)
- new net: R61.2, SW7.1
- new net: R22.2, SW3.1
- new net FAN_INA_ESP: R45.1, U14.6 (IN_A)
- new net FAN_INB_ESP: R64.1, U14.5 (IN_B)
- no-connect marks 24 -> 23
Other:
- note added: "MCP9700BT-E/TT"
- moved on the sheet: D10, D14, D15, D18, D19, D29, D3, D30, D40, D41, D5, D6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

Commit message: Completed PCB
Connections:
- net FAN_INA_ESP: now also U3.18 (IO27)
- net FAN_INB_ESP: now also U3.15 (IO28)
- net Wi-Fi_RX: now also U3.13 (IO13)
- net Wi-Fi_TX: now also U3.14 (IO14)
- no-connect marks 23 -> 21
